File: electronics/basilator.sch (KiCad schematic (older format))
At the start: 13 parts

Commit message: updated PCB
Parts:
- added U1: ESP32-PICO-D4, esp32_devkit_v2:esp32_devkit_v2, symbol RF_Module:ESP32-PICO-D4
- gave numbers to parts that had none: 13
Connections:
- new net: U1.1 (VDDA), U1.43 (VDDA), U1.46 (VDDA)
- new net: U1.25 (IO16), U1.42 (IO21)
- new net: U1.3 (VDDA3P3), U1.4 (VDDA3P3)
Changed lines of the file:
@@
 $EndDescr
 $Comp
-L power:GND #PWR?
+L power:GND #PWR04
 U 1 1 5F0F4EEE
 P 9050 2800
-F 0 "#PWR?" H 9050 2550 50  0001 C CNN
+F 0 "#PWR04" H 9050 2550 50  0001 C CNN
 F 1 "GND" H 9055 2627 50  0000 C CNN
 F 2 "" H 9050 2800 50  0001 C CNN
@@
 $EndComp
 $Comp
-L Device:LED D?
+L Device:LED D1
 U 1 1 5F0F546B
 P 9350 1400
-F 0 "D?" H 9343 1617 50  0000 C CNN
+F 0 "D1" H 9343 1617 50  0000 C CNN
 F 1 "LED" H 9343 1526 50  0000 C CNN
 F 2 "" H 9350 1400 50  0001 C CNN
@@
 $EndComp
 $Comp
-L Device:LED D?
+L Device:LED D2
 U 1 1 5F0F5FB2
 P 9350 1800
-F 0 "D?" H 9343 2017 50  0000 C CNN
+F 0 "D2" H 9343 2017 50  0000 C CNN
 F 1 "LED" H 9343 1926 50  0000 C CNN
 F 2 "" H 9350 1800 50  0001 C CNN
@@
 $EndComp
 $Comp
-L Switch:SW_SPDT_MSM SW?
+L Switch:SW_SPDT_MSM SW3
 U 1 1 5F0F272B
 P 10300 1600
-F 0 "SW?" H 10300 1885 50  0000 C CNN
+F 0 "SW3" H 10300 1885 50  0000 C CNN
 F 1 "SW_SPDT_MSM" H 10300 1794 50  0000 C CNN
 F 2 "" H 10300 1600 50  0001 C CNN
@@
 $EndComp
 $Comp
-L Switch:SW_SPDT_MSM SW?
+L Switch:SW_SPDT_MSM SW1
 U 1 1 5F0F2E32
 P 8350 2350
-F 0 "SW?" H 8350 2635 50  0000 C CNN
+F 0 "SW1" H 8350 2635 50  0000 C CNN
 F 1 "SW_SPDT_MSM" H 8350 2544 50  0000 C CNN
 F 2 "" H 8350 2350 50  0001 C CNN
@@
 Connection ~ 9050 1800
 $Comp
-L Transistor_FET:IRLB8721PBF Q?
+L Transistor_FET:IRLB8721PBF Q1
 U 1 1 5F0FB05F
 P 8950 2350
-F 0 "Q?" H 9154 2396 50  0000 L CNN
+F 0 "Q1" H 9154 2396 50  0000 L CNN
 F 1 "IRLB8721PBF" H 9154 2305 50  0000 L CNN
 F 2 "Package_TO_SOT_THT:TO-220-3_Vertical" H 9200 2275 50  0001 L CIN
@@
 	9050 2550 9050 2700
 $Comp
-L power:+12V #PWR?
+L power:+12V #PWR07
 U 1 1 5F0F486F
 P 10700 2800
-F 0 "#PWR?" H 10700 2650 50  0001 C CNN
+F 0 "#PWR07" H 10700 2650 50  0001 C CNN
 F 1 "+12V" H 10715 2973 50  0000 C CNN
 F 2 "" H 10700 2800 50  0001 C CNN
@@
 	10700 1600 10700 2800
 $Comp
-L Device:R R?
+L Device:R R3
 U 1 1 5F1074E0
 P 8750 2550
-F 0 "R?" H 8820 2596 50  0000 L CNN
+F 0 "R3" H 8820 2596 50  0000 L CNN
 F 1 "R" H 8820 2505 50  0000 L CNN
 F 2 "" V 8680 2550 50  0001 C CNN
@@
 PWM-pin
 $Comp
-L Device:R R?
+L Device:R R2
 U 1 1 5F1D63FE
 P 8150 2000
-F 0 "R?" H 8220 2046 50  0000 L CNN
+F 0 "R2" H 8220 2046 50  0000 L CNN
 F 1 "R" H 8220 1955 50  0000 L CNN
 F 2 "" V 8080 2000 50  0001 C CNN
@@
 $EndComp
 $Comp
-L Device:R R?
+L Device:R R1
 U 1 1 5F1D7DA0
 P 7850 2000
-F 0 "R?" H 7920 2046 50  0000 L CNN
+F 0 "R1" H 7920 2046 50  0000 L CNN
 F 1 "R" H 7920 1955 50  0000 L CNN
 F 2 "" V 7780 2000 50  0001 C CNN
@@
 $EndComp
 $Comp
-L power:GND #PWR?
+L power:GND #PWR03
 U 1 1 5F1E3575
 P 8300 2000
-F 0 "#PWR?" H 8300 1750 50  0001 C CNN
+F 0 "#PWR03" H 8300 1750 50  0001 C CNN
 F 1 "GND" V 8305 1872 50  0000 R CNN
 F 2 "" H 8300 2000 50  0001 C CNN
@@
 Connection ~ 8000 2000
 $Comp
-L power:+3V3 #PWR?
+L power:+3V3 #PWR01
 U 1 1 5F1E410C
 P 7700 2000
-F 0 "#PWR?" H 7700 1850 50  0001 C CNN
+F 0 "#PWR01" H 7700 1850 50  0001 C CNN
 F 1 "+3V3" V 7715 2128 50  0000 L CNN
 F 2 "" H 7700 2000 50  0001 C CNN
@@
 $EndComp
 $Comp
-L Device:D_Schottky D?
+L Device:D_Schottky D3
 U 1 1 5F1E54D6
 P 9800 1600
-F 0 "D?" H 9800 1817 50  0000 C CNN
+F 0 "D3" H 9800 1817 50  0000 C CNN
 F 1 "D_Schottky" H 9800 1726 50  0000 C CNN
 F 2 "" H 9800 1600 50  0001 C CNN
@@
 $EndComp
 $Comp
-L Transistor_FET:IRLB8721PBF Q?
+L Transistor_FET:IRLB8721PBF Q2
 U 1 1 5F1EBF23
 P 9200 4750
-F 0 "Q?" H 9404 4796 50  0000 L CNN
+F 0 "Q2" H 9404 4796 50  0000 L CNN
 F 1 "IRLB8721PBF" H 9404 4705 50  0000 L CNN
 F 2 "Package_TO_SOT_THT:TO-220-3_Vertical" H 9450 4675 50  0001 L CIN
@@
 	9300 4950 9300 5100
 $Comp
-L Device:R R?
+L Device:R R4
 U 1 1 5F1EBF2E
 P 9000 4950
-F 0 "R?" H 9070 4996 50  0000 L CNN
+F 0 "R4" H 9070 4996 50  0000 L CNN
 F 1 "R" H 9070 4905 50  0000 L CNN
 F 2 "" V 8930 4950 50  0001 C CNN
@@
 Connection ~ 9000 4750
 $Comp
-L Connector:Conn_01x02_Male J?
+L Connector:Conn_01x02_Male J1
 U 1 1 5F1F470C
 P 9850 4350
-F 0 "J?" V 9912 4394 50  0000 L CNN
+F 0 "J1" V 9912 4394 50  0000 L CNN
 F 1 "Conn_01x02_Male" V 10003 4394 50  0000 L CNN
 F 2 "" H 9850 4350 50  0001 C CNN
@@
 	9850 4550 9850 5200
 $Comp
-L power:GND #PWR?
+L power:GND #PWR05
 U 1 1 5F20141D
 P 9300 5200
-F 0 "#PWR?" H 9300 4950 50  0001 C CNN
+F 0 "#PWR05" H 9300 4950 50  0001 C CNN
 F 1 "GND" H 9305 5027 50  0000 C CNN
 F 2 "" H 9300 5200 50  0001 C CNN
@@
 	10600 4000 8900 4000
 $Comp
-L Switch:SW_SPDT_MSM SW?
+L Switch:SW_SPDT_MSM SW2
 U 1 1 5F20CF64
 P 8600 4750
-F 0 "SW?" H 8600 5035 50  0000 C CNN
+F 0 "SW2" H 8600 5035 50  0000 C CNN
 F 1 "SW_SPDT_MSM" H 8600 4944 50  0000 C CNN
 F 2 "" H 8600 4750 50  0001 C CNN
@@
 	8250 4650 8400 4650
 $Comp
-L power:+3V3 #PWR?
+L power:+3V3 #PWR02
 U 1 1 5F2228D9
 P 8250 4650
-F 0 "#PWR?" H 8250 4500 50  0001 C CNN
+F 0 "#PWR02" H 8250 4500 50  0001 C CNN
 F 1 "+3V3" H 8265 4823 50  0000 C CNN
 F 2 "" H 8250 4650 50  0001 C CNN
@@
 $EndComp
 $Comp
-L power:+5V #PWR?
+L power:+5V #PWR06
 U 1 1 5F228461
 P 9850 5200
-F 0 "#PWR?" H 9850 5050 50  0001 C CNN
+F 0 "#PWR06" H 9850 5050 50  0001 C CNN
 F 1 "+5V" H 9865 5373 50  0000 C CNN
 F 2 "" H 9850 5200 50  0001 C CNN
@@
 Text Notes 8650 3850 0    197  ~ 0
 pump-module
+$Comp
+L RF_Module:ESP32-PICO-D4 U1
+U 1 1 5FB1C90E
+P 6050 3600
+F 0 "U1" H 6050 1911 50  0000 C CNN
+F 1 "ESP32-PICO-D4" H 6050 1820 50  0000 C CNN
+F 2 "esp32_devkit_v2:esp32_devkit_v2" H 6050 1900 50  0001 C CNN
+F 3 "https://www.espressif.com/sites/default/files/documentation/esp32-pico-d4_datasheet_en.pdf" H 6300 2600 50  0001 C CNN
+	1    6050 3600
+	1    0    0    -1
+$EndComp
+Wire Wire Line
+	5250 3600 3650 3600
+Wire Wire Line
+	3650 3600 3650 5850
+Wire Wire Line
+	3650 5850 7400 5850
+Wire Wire Line
+	7400 5850 7400 3800
+Wire Wire Line
+	7400 3800 6850 3800
 $EndSCHEMATC
